File: keyring_beerclock.kicad_pcb (KiCad board)
At the start: 2 copper layers, 21.5 x 17.5 mm, 39 parts, among them J1 +BAT, J2 -BAT, J3 VCC, J4 UDPI, J5 GND, J6 +PIEZO, J7 -PIEZO, J8 USB_C_Receptacle_USB2.0, SW1 PWR_SEL, SW2 BTN_LEFT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

Commit message: Starting fresh
Parts:
- C10, C3, C4, C7, C8, J3, J4, J5, R1, R10, R11, R3, R4, R5, R6, R7, R8, R9, SW2, SW3, SW4: moved to F.Cu
- moved R5 61.4 mm to (197.8, 76.4), turned to 0 degrees
- moved R6 57.6 mm to (197.8, 71.7)
- moved R7 56.3 mm to (197.4, 81.5)
- moved SW4 56.0 mm to (192.3, 81.0), turned to 0 degrees
- moved J5 55.7 mm to (170.6, 71.2), turned to 0 degrees
- moved SW3 55.2 mm to (192.3, 76.7), turned to 0 degrees
- moved SW2 51.9 mm to (192.3, 71.6), turned to 0 degrees
- moved J4 49.7 mm to (171.0, 76.3), turned to 0 degrees
- moved R8 46.9 mm to (192.8, 121.3), turned to 0 degrees
- moved R9 45.2 mm to (192.3, 116.4), turned to 0 degrees
- moved J3 43.4 mm to (169.7, 80.8), turned to 0 degrees
- moved R3 42.8 mm to (188.4, 102.5), turned to 0 degrees
- moved R4 41.3 mm to (188.4, 104.0), turned to 0 degrees
- moved C9 38.7 mm to (188.4, 100.3)
- moved U1 37.8 mm to (191.4, 101.8)
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Connections:
- SW1 pad 1: VCC -> /BAT+
- SW1 pad 3: /BAT+ -> VCC
Routing:
- net +3V3: track 71.0 -> 0.00 mm, vias 3 -> 0
- net /BAT+: track 27.6 -> 0.00 mm, vias 2 -> 0
- net UDPI: track 18.2 -> 0.00 mm, vias 1 -> 0
- net GND: track 17.0 -> 0.00 mm, vias 9 -> 0
- net /VBUS: track 16.5 -> 0.00 mm, vias 1 -> 0
- net /-Piezo: track 16.3 -> 0.00 mm, vias 1 -> 0
- net VCC: track 14.5 -> 0.00 mm, vias 1 -> 0
- net /PWR_IN: track 14.3 -> 0.00 mm, vias 1 -> 0
- net SENSE: track 12.0 -> 0.00 mm, vias 1 -> 0
- net SCL: track 11.6 -> 0.00 mm, vias 1 -> 0
- net SDA: track 11.3 -> 0.00 mm, vias 1 -> 0
- net BTN_RIGHT: track 10.0 -> 0.00 mm, vias 1 -> 0
- net BTN_MID: track 9.29 -> 0.00 mm, vias 1 -> 0
- net BTN_LEFT: track 7.23 -> 0.00 mm, vias 1 -> 0
- net /VBAT: track 7.11 -> 0.00 mm
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- removed copper zone on B.Cu, net GND
- removed copper zone on F.Cu, net GND
Other:
- board outline removed
- board text removed: "BAT"
- board text removed: "Feb 23"
- board text removed: "G"
- board text removed: "GND"
- board text removed: "P+"
- board text removed: "P-"
- board text removed: "U"
- board text removed: "V"
- board text removed: "V1.0"

Commit message: Finished layout, ready to order
Parts:
- removed R5, R6: 2K, Resistor_SMD:R_0402_1005Metric_Pad0.72x0.64mm_HandSolder
- removed SW2: BTN_LEFT, Button_Switch_SMD:SW_SPST_B3U-1000P
- removed SW4: BTN_MID, Button_Switch_SMD:SW_SPST_B3U-1000P
- R7, SW3, U1: moved to B.Cu
- moved R8 68.8 mm to (148.2, 68.9), turned to 90 degrees
- moved R7 68.2 mm to (130.4, 68.8), turned to 90 degrees
- moved U1 64.3 mm to (132.2, 76.6), turned to 180 degrees
- moved R9 64.1 mm to (149.3, 68.9), turned to -90 degrees
- moved J7 63.0 mm to (153.3, 68.1), turned to 90 degrees
- moved SW3 59.4 mm to (133.4, 69.3), turned to 180 degrees
- moved R4 58.7 mm to (141.5, 68.7), turned to -90 degrees
- moved R2 58.5 mm to (142.6, 68.7), turned to 90 degrees
- moved J6 58.4 mm to (153.3, 70.7), turned to 90 degrees
- moved C5 58.3 mm to (143.7, 68.7), turned to 90 degrees
- moved C6 58.1 mm to (144.8, 68.7), turned to 90 degrees
- moved R3 53.5 mm to (141.5, 76.8), turned to 90 degrees
- moved C9 51.5 mm to (142.6, 76.8), turned to -90 degrees
- moved U4 50.4 mm to (143.0, 72.7), turned to 180 degrees
- moved C2 49.9 mm to (143.7, 76.8), turned to 90 degrees
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Connections:
- U4 pad 17: BTN_MID -> unconnected-(U4-Pad17)
- U4 pad 18: BTN_LEFT -> unconnected-(U4-Pad18)
Routing:
- net BTN_RIGHT: track 0.00 -> 21.8 mm, vias 0 -> 2
- net +3V3: track 0.00 -> 20.3 mm, vias 0 -> 8
- net /BAT+: track 0.00 -> 19.9 mm
- net /PWR_IN: track 0.00 -> 17.3 mm, vias 0 -> 2
- net /C2N: track 0.00 -> 17.1 mm, vias 0 -> 1
- net /C2P: track 0.00 -> 17.0 mm, vias 0 -> 1
- net /VCC_CAP: track 0.00 -> 16.6 mm, vias 0 -> 1
- net SDA: track 0.00 -> 15.9 mm, vias 0 -> 1
- net /VCOMM: track 0.00 -> 15.2 mm, vias 0 -> 1
- net /C1P: track 0.00 -> 14.7 mm, vias 0 -> 1
- net /C1N: track 0.00 -> 14.4 mm, vias 0 -> 1
- net SCL: track 0.00 -> 14.3 mm, vias 0 -> 1
- net /VBUS: track 0.00 -> 14.0 mm
- net /IREF: track 0.00 -> 13.5 mm, vias 0 -> 1
- net /VBAT: track 0.00 -> 12.8 mm, vias 0 -> 1
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- added copper zone on In2.Cu, net +3V3
- added copper zone on B.Cu, net GND
- added copper zone on F.Cu, net GND
- added copper zone on In1.Cu, net GND
Other:
- board outline added: 25.4 x 15.4 mm
- copper layers 2 -> 4
- board text added: "Adler2023"
- board text added: "B+"
- board text added: "B-"
- board text added: "G"
- board text added: "P+"
- board text added: "P-"
- board text added: "U"
- board text added: "V"
- board text added: "V1"
